File: Moriduino.sch (KiCad schematic (older format))
At the start: 42 parts, among them CN1 CON_USB-C-16, CN2 CON_AVRISP, J1 USB_B, J2 Barrel_Jack_Switch, P1 Power, P2 Analog, P3 Digital, P4 Digital, P5 CONN_01X01, P6 CONN_01X01, P7 CONN_01X01, P8 CONN_01X01, Q1 FDN340P, U1 AP1117-50, U2 LMV358, U3 IC_FT232RQ, U4 ATmega328P-PU, U5 LDO_5p_NJM2865, Y1 16MHz

Commit message: 配線を少し進めた
Connections:
- net GND: now also U1.1 (GND)
Changed lines of the file:
@@
 Wire Wire Line
 	9050 1700 9050 1350
+$Comp
+L power:GND #PWR?
+U 1 1 5EC2A9AC
+P 2200 6750
+F 0 "#PWR?" H 2200 6500 50  0001 C CNN
+F 1 "GND" H 2205 6577 50  0000 C CNN
+F 2 "" H 2200 6750 50  0001 C CNN
+F 3 "" H 2200 6750 50  0001 C CNN
+	1    2200 6750
+	1    0    0    -1
+$EndComp
+Wire Wire Line
+	2200 6750 2200 6500
 $EndSCHEMATC

Commit message: 一通り完成
Connections:
- net +5V: now also D2.2 (A), D3.2 (A)
- net GND: now also CN1.FG, J2.2, U3.33 (GND(e)); no longer J2.1
- net at D5.2 (A): now also J2.1; no longer J2.2
Changed lines of the file:
@@
 F 3 "~" H 1150 6260 50  0001 C CNN
 	1    1100 6300
-	1    0    0    1
+	1    0    0    -1
 $EndComp
 $Comp
@@
 L power:GND #PWR016
 U 1 1 5EC57963
-P 3400 3650
-F 0 "#PWR016" H 3400 3400 50  0001 C CNN
-F 1 "GND" H 3405 3477 50  0000 C CNN
-F 2 "" H 3400 3650 50  0001 C CNN
-F 3 "" H 3400 3650 50  0001 C CNN
-	1    3400 3650
-	1    0    0    -1
-$EndComp
-Wire Wire Line
-	3400 3150 3400 3650
+P 3350 3650
+F 0 "#PWR016" H 3350 3400 50  0001 C CNN
+F 1 "GND" H 3355 3477 50  0000 C CNN
+F 2 "" H 3350 3650 50  0001 C CNN
+F 3 "" H 3350 3650 50  0001 C CNN
+	1    3350 3650
+	1    0    0    -1
+$EndComp
 Wire Wire Line
 	3150 3350 3150 3650
@@
 Wire Wire Line
 	1400 6400 1450 6400
-Wire Wire Line
-	1450 6400 1450 6750
-Wire Wire Line
-	1400 6200 1600 6200
 $Comp
 L Device:R R5
@@
 	1700 4950 1750 4950
 Connection ~ 1750 4950
-Wire Wire Line
-	1750 4950 1750 5150
 $Comp
 L Device:R R4
@@
 	9050 1700 9050 1350
 $Comp
-L power:GND #PWR?
+L power:GND #PWR0101
 U 1 1 5EC2A9AC
 P 2200 6750
-F 0 "#PWR?" H 2200 6500 50  0001 C CNN
+F 0 "#PWR0101" H 2200 6500 50  0001 C CNN
 F 1 "GND" H 2205 6577 50  0000 C CNN
 F 2 "" H 2200 6750 50  0001 C CNN
@@
 Wire Wire Line
 	2200 6750 2200 6500
+Wire Wire Line
+	1400 6200 1600 6200
+Wire Wire Line
+	1450 6400 1450 6750
+Wire Wire Line
+	3400 3150 3350 3150
+Wire Wire Line
+	3350 3150 3350 3350
+Wire Wire Line
+	3400 3350 3350 3350
+Connection ~ 3350 3350
+Wire Wire Line
+	3350 3350 3350 3650
+$Comp
+L power:+5V #PWR0102
+U 1 1 5ECE3471
+P 5350 2300
+F 0 "#PWR0102" H 5350 2150 50  0001 C CNN
+F 1 "+5V" H 5365 2473 50  0000 C CNN
+F 2 "" H 5350 2300 50  0001 C CNN
+F 3 "" H 5350 2300 50  0001 C CNN
+	1    5350 2300
+	1    0    0    -1
+$EndComp
+Wire Wire Line
+	5350 2300 5350 2400
+Wire Wire Line
+	5350 2400 5350 2550
+Connection ~ 5350 2400
+Wire Wire Line
+	1750 4950 1750 5050
+Wire Wire Line
+	1700 5050 1750 5050
+Connection ~ 1750 5050
+Wire Wire Line
+	1750 5050 1750 5150
 $EndSCHEMATC

Commit message: 配線ミスを修正しベタGNDを追加
Connections:
- net GND: now also D4.1 (K)
Changed lines of the file:
@@
 Wire Wire Line
 	1750 5050 1750 5150
+Wire Wire Line
+	9900 4750 9900 4800
 $EndSCHEMATC

Commit message: pMOSの向きが逆だったのを修正
Connections:
- net +5V: now also Q1.3 (D); no longer Q1.2 (S)
- net at F1.1: now also Q1.2 (S); no longer Q1.3 (D)
Changed lines of the file:
@@
 F 5 "305030026" H 2330 2800 20  0001 C CNN "SKU"
 	1    2300 2650
-	0    -1   1    0
+	0    1    1    0
 $EndComp
 $Comp
@@
 Wire Wire Line
 	1450 2650 1650 2650
-Wire Wire Line
-	1950 2650 2100 2650
 $Comp
 L power:+5V #PWR011
@@
 $EndComp
 Wire Wire Line
-	2500 2650 2550 2650
-Wire Wire Line
 	2050 1650 2300 1650
-Wire Wire Line
-	2300 1650 2300 2450
 $Comp
 L power:+3.3V #PWR07
@@
 Wire Wire Line
 	9900 4750 9900 4800
+Wire Wire Line
+	2100 2650 1950 2650
+Wire Wire Line
+	2500 2650 2550 2650
+Wire Wire Line
+	2300 2450 2300 1650
 $EndSCHEMATC
